File: examples/1x4-rotations-90-step/keyboard-after.kicad_pcb (KiCad board)
At the start: 2 copper layers, 81.2 x 24 mm, 8 parts, among them SW1 SW_Push, SW2 SW_Push, SW3 SW_Push, SW4 SW_Push

Commit message: Update examples kicad files
Other:
- board outline removed
- net class Default removed

Commit message: Maintain own copy of footprints used in examples
Because testing with more footprints variants will be added soon,
it would be easier to maintain own copy of used footprints than
include multiple submodules for various libraries.
Parts:
- SW1, SW2, SW3, SW4: footprint Switch_Keyboard_Cherry_MX:SW_Cherry_MX_PCB_1.00u -> examples:SW_Cherry_MX_PCB_1.00u
Changed lines of the file:
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@@
   (net 8 "N$4")
   (net 9 "ROW0")
-  (footprint "Switch_Keyboard_Cherry_MX:SW_Cherry_MX_PCB_1.00u" (layer "F.Cu")
+  (footprint "examples:SW_Cherry_MX_PCB_1.00u" (layer "F.Cu")
     (at 34.525 34.525)
     (descr "Cherry MX keyswitch, https://www.cherrymx.de/en/dev.html")
@@
     )
   )
-  (footprint "Switch_Keyboard_Cherry_MX:SW_Cherry_MX_PCB_1.00u" (layer "F.Cu")
+  (footprint "examples:SW_Cherry_MX_PCB_1.00u" (layer "F.Cu")
     (at 53.575 34.525 -90)
     (descr "Cherry MX keyswitch, https://www.cherrymx.de/en/dev.html")
@@
     )
   )
-  (footprint "Switch_Keyboard_Cherry_MX:SW_Cherry_MX_PCB_1.00u" (layer "F.Cu")
+  (footprint "examples:SW_Cherry_MX_PCB_1.00u" (layer "F.Cu")
     (at 72.625 34.525 180)
     (descr "Cherry MX keyswitch, https://www.cherrymx.de/en/dev.html")
@@
     )
   )
-  (footprint "Switch_Keyboard_Cherry_MX:SW_Cherry_MX_PCB_1.00u" (layer "F.Cu")
+  (footprint "examples:SW_Cherry_MX_PCB_1.00u" (layer "F.Cu")
     (at 91.675 34.525 90)
     (descr "Cherry MX keyswitch, https://www.cherrymx.de/en/dev.html")
