File: examples/2x2/keyboard-after.kicad_pcb (KiCad board)
At the start: 2 copper layers, 43.1 x 43.1 mm, 8 parts, among them SW1 SW_Push, SW2 SW_Push, SW3 SW_Push, SW4 SW_Push

Commit message: Update examples kicad files
Parts:
- D1, D2, D3, D4: footprint D_SOD-323F -> Diode_SMD:D_SOD-323F
- SW1, SW2, SW3, SW4: footprint SW_Cherry_MX_PCB_1.00u -> Switch_Keyboard_Cherry_MX:SW_Cherry_MX_PCB_1.00u
Other:
- board outline removed
- net class Default removed

Commit message: Maintain own copy of footprints used in examples
Because testing with more footprints variants will be added soon,
it would be easier to maintain own copy of used footprints than
include multiple submodules for various libraries.
Parts:
- SW1, SW2, SW3, SW4: footprint Switch_Keyboard_Cherry_MX:SW_Cherry_MX_PCB_1.00u -> examples:SW_Cherry_MX_PCB_1.00u
Changed lines of the file:
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@@
   (net 7 "COL0")
   (net 8 "COL1")
-  (footprint "Switch_Keyboard_Cherry_MX:SW_Cherry_MX_PCB_1.00u" (layer "F.Cu")
+  (footprint "examples:SW_Cherry_MX_PCB_1.00u" (layer "F.Cu")
     (at 34.525 34.525)
     (descr "Cherry MX keyswitch, https://www.cherrymx.de/en/dev.html")
@@
     )
   )
-  (footprint "Switch_Keyboard_Cherry_MX:SW_Cherry_MX_PCB_1.00u" (layer "F.Cu")
+  (footprint "examples:SW_Cherry_MX_PCB_1.00u" (layer "F.Cu")
     (at 53.575 34.525)
     (descr "Cherry MX keyswitch, https://www.cherrymx.de/en/dev.html")
@@
     )
   )
-  (footprint "Switch_Keyboard_Cherry_MX:SW_Cherry_MX_PCB_1.00u" (layer "F.Cu")
+  (footprint "examples:SW_Cherry_MX_PCB_1.00u" (layer "F.Cu")
     (at 34.525 53.575)
     (descr "Cherry MX keyswitch, https://www.cherrymx.de/en/dev.html")
@@
     )
   )
-  (footprint "Switch_Keyboard_Cherry_MX:SW_Cherry_MX_PCB_1.00u" (layer "F.Cu")
+  (footprint "examples:SW_Cherry_MX_PCB_1.00u" (layer "F.Cu")
     (at 53.575 53.575)
     (descr "Cherry MX keyswitch, https://www.cherrymx.de/en/dev.html")
