File: examples/2x3-rotations/keyboard-before.kicad_pcb (KiCad board)
At the start: 2 copper layers, 11 parts, among them SW1 SW_Push, SW2 SW_Push, SW3 SW_Push, SW4 SW_Push, SW5 SW_Push

Commit message: Update examples kicad files
Other:
- net class Default removed

Commit message: Maintain own copy of footprints used in examples
Because testing with more footprints variants will be added soon,
it would be easier to maintain own copy of used footprints than
include multiple submodules for various libraries.
Parts:
- ST3: footprint Mounting_Keyboard_Stabilizer:Stabilizer_Cherry_MX_2u -> examples:Stabilizer_Cherry_MX_2u
- SW1, SW2, SW4, SW5: footprint Switch_Keyboard_Cherry_MX:SW_Cherry_MX_PCB_1.00u -> examples:SW_Cherry_MX_PCB_1.00u
- SW3: footprint Switch_Keyboard_Cherry_MX:SW_Cherry_MX_PCB_2.00u -> examples:SW_Cherry_MX_PCB_2.00u
Changed lines of the file:
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@@
     )
   )
-  (footprint "Mounting_Keyboard_Stabilizer:Stabilizer_Cherry_MX_2u" (layer "F.Cu")
+  (footprint "examples:Stabilizer_Cherry_MX_2u" (layer "F.Cu")
     (at 12.306899 -12.216001)
     (descr "Cherry MX key stabilizer 2u 2.25u 2.5u 2.75u")
@@
     )
   )
-  (footprint "Switch_Keyboard_Cherry_MX:SW_Cherry_MX_PCB_1.00u" (layer "F.Cu")
+  (footprint "examples:SW_Cherry_MX_PCB_1.00u" (layer "F.Cu")
     (at 67.3 -31.3)
     (descr "Cherry MX keyswitch, https://www.cherrymx.de/en/dev.html")
@@
     )
   )
-  (footprint "Switch_Keyboard_Cherry_MX:SW_Cherry_MX_PCB_1.00u" (layer "F.Cu")
+  (footprint "examples:SW_Cherry_MX_PCB_1.00u" (layer "F.Cu")
     (at 56.96 -11.15)
     (descr "Cherry MX keyswitch, https://www.cherrymx.de/en/dev.html")
@@
     )
   )
-  (footprint "Switch_Keyboard_Cherry_MX:SW_Cherry_MX_PCB_2.00u" (layer "F.Cu")
+  (footprint "examples:SW_Cherry_MX_PCB_2.00u" (layer "F.Cu")
     (at 17.475 -31.3)
     (descr "Cherry MX keyswitch, https://www.cherrymx.de/en/dev.html")
@@
     )
   )
-  (footprint "Switch_Keyboard_Cherry_MX:SW_Cherry_MX_PCB_1.00u" (layer "F.Cu")
+  (footprint "examples:SW_Cherry_MX_PCB_1.00u" (layer "F.Cu")
     (at 47.15 -31.3)
     (descr "Cherry MX keyswitch, https://www.cherrymx.de/en/dev.html")
@@
     )
   )
-  (footprint "Switch_Keyboard_Cherry_MX:SW_Cherry_MX_PCB_1.00u" (layer "F.Cu")
+  (footprint "examples:SW_Cherry_MX_PCB_1.00u" (layer "F.Cu")
     (at 36.81 -11.15)
     (descr "Cherry MX keyswitch, https://www.cherrymx.de/en/dev.html")
