File: examples/3x2-sizes/keyboard-before.kicad_pcb (KiCad board)
At the start: 2 copper layers, 12 parts, among them SW1 SW_Push, SW2 SW_Push, SW3 SW_Push, SW4 SW_Push, SW5 SW_Push, SW6 SW_Push

Commit message: Update examples kicad files
Other:
- net class Default removed

Commit message: Maintain own copy of footprints used in examples
Because testing with more footprints variants will be added soon,
it would be easier to maintain own copy of used footprints than
include multiple submodules for various libraries.
Parts:
- SW1, SW2, SW4, SW6: footprint Switch_Keyboard_Cherry_MX:SW_Cherry_MX_PCB_1.00u -> examples:SW_Cherry_MX_PCB_1.00u
- SW3: footprint Switch_Keyboard_Cherry_MX:SW_Cherry_MX_PCB_1.50u -> examples:SW_Cherry_MX_PCB_1.50u
- SW5: footprint Switch_Keyboard_Cherry_MX:SW_Cherry_MX_PCB_1.75u -> examples:SW_Cherry_MX_PCB_1.75u
Changed lines of the file:
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@@
     )
   )
-  (footprint "Switch_Keyboard_Cherry_MX:SW_Cherry_MX_PCB_1.00u" (layer "F.Cu")
+  (footprint "examples:SW_Cherry_MX_PCB_1.00u" (layer "F.Cu")
     (at 57.77 -11.55)
     (descr "Cherry MX keyswitch, https://www.cherrymx.de/en/dev.html")
@@
     )
   )
-  (footprint "Switch_Keyboard_Cherry_MX:SW_Cherry_MX_PCB_1.00u" (layer "F.Cu")
+  (footprint "examples:SW_Cherry_MX_PCB_1.00u" (layer "F.Cu")
     (at 37.62 -11.55)
     (descr "Cherry MX keyswitch, https://www.cherrymx.de/en/dev.html")
@@
     )
   )
-  (footprint "Switch_Keyboard_Cherry_MX:SW_Cherry_MX_PCB_1.50u" (layer "F.Cu")
+  (footprint "examples:SW_Cherry_MX_PCB_1.50u" (layer "F.Cu")
     (at 12.7125 -11.55)
     (descr "Cherry MX keyswitch, https://www.cherrymx.de/en/dev.html")
@@
     )
   )
-  (footprint "Switch_Keyboard_Cherry_MX:SW_Cherry_MX_PCB_1.00u" (layer "F.Cu")
+  (footprint "examples:SW_Cherry_MX_PCB_1.00u" (layer "F.Cu")
     (at 42.38 -31.7)
     (descr "Cherry MX keyswitch, https://www.cherrymx.de/en/dev.html")
@@
     )
   )
-  (footprint "Switch_Keyboard_Cherry_MX:SW_Cherry_MX_PCB_1.75u" (layer "F.Cu")
+  (footprint "examples:SW_Cherry_MX_PCB_1.75u" (layer "F.Cu")
     (at 15.09375 -31.7)
     (descr "Cherry MX keyswitch, https://www.cherrymx.de/en/dev.html")
@@
     )
   )
-  (footprint "Switch_Keyboard_Cherry_MX:SW_Cherry_MX_PCB_1.00u" (layer "F.Cu")
+  (footprint "examples:SW_Cherry_MX_PCB_1.00u" (layer "F.Cu")
     (at 62.53 -31.7)
     (descr "Cherry MX keyswitch, https://www.cherrymx.de/en/dev.html")
