File: examples/2x3-rotations-custom-diode-with-track-and-complex-footprint/diode_template.kicad_pcb (KiCad board)
At the start: 2 copper layers, 2 parts, among them SW1 SW_Push

Commit message: Fix via in connections template
Free via do not work with connection template duplication because it
won't inherit netcode after building connectivity of template PCB file.
Routing:
- net COL0: vias 0 -> 1
- net (no net): vias 1 -> 0
Changed lines of the file:
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@@
     )
   )
-  (via (at 0 -2.736) (size 0.8) (drill 0.4) (layers "F.Cu" "B.Cu") (free) (net 0))
+  (via (at 0 -2.736) (size 0.8) (drill 0.4) (layers "F.Cu" "B.Cu") (net 1))
   (segment (start 0 3.604) (end 0 5.9) (width 0.25) (layer "F.Cu") (net 1))
   (segment (start -1.2475 -2.736) (end -2.784 -1.1995) (width 0.25) (layer "F.Cu") (net 1))
